Commit message: Add files via upload

File: Vox-Bot/vox_description/urdf/voxbot.urdf (robot description, URDF)
Before this commit: robot voxbot, 49 links, 48 joints
Links:
- added link belt_moving, mass 0.1; collision box size=0.4 0.001 0.4; visual box size=0.4 0.001 0.4
- added link belt_moving_up, mass 0.1; collision box size=0.4 0.001 0.4; visual box size=0.4 0.001 0.4
- added link conv_link, mass 0.1; collision box size=0.4 0.01 0.4; visual box size=0.4 0.01 0.4
- added link conv_link_up, mass 0.1; collision box size=0.4 0.01 0.4; visual box size=0.4 0.01 0.4
- link base_link: mass 0.465033072874443 -> 13.465033072874443
Joints:
- added joint belt_joint: type prismatic, parent conv_link, child belt_moving, origin xyz=0.0 -0.005 0.0 rpy=0.0 0.0 0.0, axis 0 0 1, limit lower=0.0 upper=0.7 effort=100000000 velocity=100000
- added joint belt_joint_up: type fixed, parent belt_moving, child belt_moving_up, origin xyz=0.0 -0.19 0.0 rpy=0.0 0.0 0.0
- added joint conv_joint: type fixed, parent base_link, child conv_link, origin xyz=-0.1 -0.1414 -0.1 rpy=0.785 0.785 0
- added joint conv_joint_up: type fixed, parent conv_link, child conv_link_up, origin xyz=0 -0.2 0 rpy=0 0 0
- joint cube_joint: origin xyz=0 -0.3 0 rpy=1.57 -0.785 0 -> xyz=0 -0.65 0 rpy=1.57 -0.785 0
